Commit message: First link and joint

File: assets/claw.urdf (robot description, URDF)
Before this commit: robot planar_claw, 0 links, 0 joints
Links:
- added link base_link
- added link left_link_1; visual box size=0.02 0.10 0.02
- added link right_link_1; visual box size=0.02 0.10 0.02
Joints:
- added joint left_joint_1: type revolute, parent base_link, child left_link_1, origin xyz=0 0 0, axis 0 0 1, limit lower=-1.5708 upper=1.5708 effort=10 velocity=2
- added joint right_joint_1: type revolute, parent base_link, child right_link_1, origin xyz=0 0 0, axis 0 0 1, limit lower=-1.5708 upper=1.5708 effort=10 velocity=2

Commit message: Including collision geometry

File: assets/claw.urdf (robot description, URDF)
Before this commit: robot planar_claw, 3 links, 2 joints
Links:
- added link left_link_2; collision box size=0.10 0.02 0.02; visual box size=0.10 0.02 0.02
- added link left_link_3; collision box size=0.10 0.02 0.02; visual box size=0.10 0.02 0.02
- added link right_link_2; collision box size=0.10 0.02 0.02; visual box size=0.10 0.02 0.02
- added link right_link_3; collision box size=0.10 0.02 0.02; visual box size=0.10 0.02 0.02
- link left_link_1: geometry collision box size=0.10 0.02 0.02; visual box size=0.10 0.02 0.02
- link right_link_1: geometry collision box size=0.10 0.02 0.02; visual box size=0.10 0.02 0.02
Joints:
- added joint left_joint_2: type revolute, parent left_link_1, child left_link_2, origin xyz=-0.10 0 0, axis 0 0 1, limit lower=-1.5708 upper=1.5708 effort=10 velocity=2
- added joint left_joint_3: type revolute, parent left_link_2, child left_link_3, origin xyz=-0.10 0 0, axis 0 0 1, limit lower=-1.5708 upper=1.5708 effort=10 velocity=2
- added joint right_joint_2: type revolute, parent right_link_1, child right_link_2, origin xyz=0.10 0 0, axis 0 0 1, limit lower=-1.5708 upper=1.5708 effort=10 velocity=2
- added joint right_joint_3: type revolute, parent right_link_2, child right_link_3, origin xyz=0.10 0 0, axis 0 0 1, limit lower=-1.5708 upper=1.5708 effort=10 velocity=2

Commit message: Added mass and inertia

File: assets/claw.urdf (robot description, URDF)
Before this commit: robot planar_claw, 7 links, 6 joints
Links:
- link left_link_1: mass None -> 0.06
- link left_link_2: mass None -> 0.06
- link left_link_3: mass None -> 0.06
- link right_link_1: mass None -> 0.06
- link right_link_2: mass None -> 0.06
- link right_link_3: mass None -> 0.06

Commit message: Checkpoint save

File: assets/claw.urdf (robot description, URDF)
Before this commit: robot planar_claw, 7 links, 6 joints
Links:
- link base_link: mass None -> 1.0

File: assets/plane.urdf (robot description, URDF)
Before this commit: robot plane, 1 links, 0 joints
Links:
- link plane_link: mass None -> 1.0

Commit message: Change axis to z=0

File: assets/claw.urdf (robot description, URDF)
Before this commit: robot planar_claw, 7 links, 6 joints
Links:
- link left_link_1: geometry collision box size=0.02 0.02 0.09; visual box size=0.02 0.02 0.09
- link left_link_2: geometry collision box size=0.02 0.02 0.09; visual box size=0.02 0.02 0.09
- link left_link_3: geometry collision box size=0.02 0.02 0.09; visual box size=0.02 0.02 0.09
- link right_link_1: geometry collision box size=0.02 0.02 0.09; visual box size=0.02 0.02 0.09
- link right_link_2: geometry collision box size=0.02 0.02 0.09; visual box size=0.02 0.02 0.09
- link right_link_3: geometry collision box size=0.02 0.02 0.09; visual box size=0.02 0.02 0.09
Joints:
- joint left_joint_1: axis 0 0 1 -> 1 0 0; limit lower=-1.5708 upper=1.5708 effort=10 velocity=2 -> lower=-1.5708 upper=1.5708 effort=2 velocity=2; origin xyz=0 0 0 -> xyz=0 -0.03 0
- joint left_joint_2: axis 0 0 1 -> 1 0 0; limit lower=-1.5708 upper=1.5708 effort=10 velocity=2 -> lower=-1.5708 upper=1.5708 effort=2 velocity=2; origin xyz=-0.10 0 0 -> xyz=0 0 -0.09
- joint left_joint_3: axis 0 0 1 -> 1 0 0; limit lower=-1.5708 upper=1.5708 effort=10 velocity=2 -> lower=-1.5708 upper=1.5708 effort=2 velocity=2; origin xyz=-0.10 0 0 -> xyz=0 0 -0.09
- joint right_joint_1: axis 0 0 1 -> 1 0 0; limit lower=-1.5708 upper=1.5708 effort=10 velocity=2 -> lower=-1.5708 upper=1.5708 effort=2 velocity=2; origin xyz=0 0 0 -> xyz=0 0.03 0
- joint right_joint_2: axis 0 0 1 -> 1 0 0; limit lower=-1.5708 upper=1.5708 effort=10 velocity=2 -> lower=-1.5708 upper=1.5708 effort=2 velocity=2; origin xyz=0.10 0 0 -> xyz=0 0 -0.09
- joint right_joint_3: axis 0 0 1 -> 1 0 0; limit lower=-1.5708 upper=1.5708 effort=10 velocity=2 -> lower=-1.5708 upper=1.5708 effort=2 velocity=2; origin xyz=0.10 0 0 -> xyz=0 0 -0.09

File: assets/cube.urdf (robot description, URDF)
Before this commit: robot cube, 1 links, 0 joints
Links:
- added link cube_mount, mass 1.0
- added link cube_slider_y_link, mass 0.0001
- added link cube_slider_z_link, mass 0.0001
- link cube_link: geometry collision box size=0.02 0.08 0.08; visual box size=0.02 0.08 0.08
Joints:
- added joint cube_joint_x: type continuous, parent cube_slider_z_link, child cube_link, origin xyz=0 0 0, axis 1 0 0, limit effort=1000 velocity=100
- added joint cube_slider_y: type prismatic, parent cube_mount, child cube_slider_y_link, origin xyz=0 0 0, axis 0 1 0, limit lower=-0.4 upper=0.4 effort=1000 velocity=10
- added joint cube_slider_z: type prismatic, parent cube_slider_y_link, child cube_slider_z_link, origin xyz=0 0 0, axis 0 0 1, limit lower=-0.05 upper=0.5 effort=1000 velocity=10
