Commit message: Use a nonlinear negative reward for angular error

File: assets/cube.urdf (robot description, URDF)
Before this commit: robot cube, 4 links, 3 joints
Links:
- link cube_link: geometry collision box size=0.02 0.06 0.10; visual box size=0.02 0.06 0.10

Commit message: Lower claw base so fingertips can reach the floor

File: assets/cube.urdf (robot description, URDF)
Before this commit: robot cube, 4 links, 3 joints
Links:
- link cube_link: geometry collision box size=0.02 0.07 0.09; visual box size=0.02 0.07 0.09

Commit message: Lower claw base and widen cube for easier recovery

File: assets/cube.urdf (robot description, URDF)
Before this commit: robot cube, 4 links, 3 joints
Links:
- link cube_link: geometry collision box size=0.02 0.08 0.09; visual box size=0.02 0.08 0.09
